File: Project/button-debouncer.kicad_sch (KiCad schematic)
At the start: 0 parts

Commit message: schematics done
Parts:
- added C1, C2, C3, C4, C5, C6, C7, C8, C9: 1u, symbol Device:C
- added D1, D2, D3, D4: LED, symbol Device:LED
- added H1, H2, H3, H4: MountingHole_Pad, symbol Mechanical:MountingHole_Pad
- added J1, J2, J3, J4: Conn_01x02, symbol Connector_Generic:Conn_01x02
- added J5: Conn_01x06, symbol Connector_Generic:Conn_01x06
- added R1, R10, R11, R12, R2, R3, R4, R5, R6, R7, R8, R9: R, symbol Device:R
- added SW1, SW2, SW4, SW5: SW_Push, symbol Switch:SW_Push
- added SW3, SW6: SW_SPDT, symbol Switch:SW_SPDT
- added U1: 40106, symbol 4xxx:40106
- added U2: SN74HCS32, symbol 74xx:74LS32
Connections:
- new net: R12.1, U2.11
- new net: R10.1, U2.6
- new net: D2.2 (A), R10.2
- new net: C5.1, R3.2, R4.2, U1.3
- new net: C6.1, R5.2, R6.2, U1.5
- new net: SW3.3 (C), U1.6, U1.9
- new net: R1.1, SW1.2
- new net: C3.1, R1.2, R2.2, U1.1
- new net: SW6.1 (A), U1.12
- new net: SW6.3 (C), U1.10, U1.13
- new net: R11.1, U2.8
- new net: C7.1, R7.2, R8.2, U1.11
- new net: D3.2 (A), R11.2
- new net: R7.1, SW5.2
- new net: R5.1, SW4.2
- new net: D1.2 (A), R9.2
- new net: SW3.1 (A), U1.8
- new net: R9.1, U2.3
- new net: D4.2 (A), R12.2
- new net: R3.1, SW2.2
- new net +5V: C1.1, C2.1, C4.1, C8.1, C9.1, J1.1 (Pin_1), J1.2 (Pin_2), J2.1 (Pin_1), J2.2 (Pin_2), J5.1 (Pin_1), R2.1, R4.1, R6.1, R8.1, U1.14 (VDD), U2.14 (VCC)
- new net GND: C1.2, C2.2, C3.2, C4.2, C5.2, C6.2, C7.2, C8.2, C9.2, D1.1 (K), D2.1 (K), D3.1 (K), D4.1 (K), H1.1, H2.1, H3.1, H4.1, J3.1 (Pin_1), J3.2 (Pin_2), J4.1 (Pin_1), J4.2 (Pin_2), J5.6 (Pin_6), SW1.1, SW2.1, SW4.1, SW5.1, U1.7 (VSS), U2.7 (GND)
- new net Q1: J5.2 (Pin_2), U1.2, U2.1, U2.2
- new net Q2: J5.3 (Pin_3), U1.4, U2.4, U2.5
- new net Q3: J5.4 (Pin_4), SW3.2 (B), U2.10, U2.9
- new net Q4: J5.5 (Pin_5), SW6.2 (B), U2.12, U2.13
Other:
- note added: "BUTTON DEBOUNCERS"
- note added: "ICs Power Supply"
- note added: "IO PINS"
- note added: "LED INDICATORS"
- note added: "MOUNTING HOLES"

Commit message: fixed power flags
Parts:
- renumbered C4 to C3, C8 to C4, C3 to C5, C5 to C6, C6 to C7, C7 to C8
Changed lines of the file:
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@@
   (junction (at 45.72 57.15) (diameter 0) (color 0 0 0 0)
   )
+  (junction (at 96.52 30.48) (diameter 0) (color 0 0 0 0)
+  )
   (junction (at 223.52 34.29) (diameter 0) (color 0 0 0 0)
   )
@@
   (junction (at 44.45 140.97) (diameter 0) (color 0 0 0 0)
   )
+  (junction (at 96.52 58.42) (diameter 0) (color 0 0 0 0)
+  )
   (junction (at 223.52 76.2) (diameter 0) (color 0 0 0 0)
   )
@@
     (stroke (width 0) (type default))
   )
+  (wire (pts (xy 106.68 58.42) (xy 96.52 58.42))
+    (stroke (width 0) (type default))
+  )
   (wire (pts (xy 88.9 36.83) (xy 83.82 36.83))
     (stroke (width 0) (type default))
@@
     (stroke (width 0) (type default))
   )
+  (wire (pts (xy 106.68 57.15) (xy 106.68 58.42))
+    (stroke (width 0) (type default))
+  )
   (wire (pts (xy 248.92 48.26) (xy 251.46 48.26))
     (stroke (width 0) (type default))
@@
     (stroke (width 0) (type default))
   )
-  (wire (pts (xy 96.52 27.94) (xy 96.52 40.64))
+  (wire (pts (xy 96.52 27.94) (xy 96.52 30.48))
     (stroke (width 0) (type default))
   )
@@
     (stroke (width 0) (type default))
   )
+  (wire (pts (xy 96.52 30.48) (xy 96.52 40.64))
+    (stroke (width 0) (type default))
+  )
   (wire (pts (xy 110.49 96.52) (xy 115.57 96.52))
     (stroke (width 0) (type default))
@@
     (stroke (width 0) (type default))
   )
+  (wire (pts (xy 106.68 30.48) (xy 96.52 30.48))
+    (stroke (width 0) (type default))
+  )
   (wire (pts (xy 31.75 96.52) (xy 25.4 96.52))
     (stroke (width 0) (type default))
@@
     (stroke (width 0) (type default))
   )
+  (wire (pts (xy 96.52 58.42) (xy 96.52 59.69))
+    (stroke (width 0) (type default))
+  )
   (wire (pts (xy 44.45 140.97) (xy 55.88 140.97))
     (stroke (width 0) (type default))
   )
-  (wire (pts (xy 96.52 48.26) (xy 96.52 59.69))
+  (wire (pts (xy 96.52 48.26) (xy 96.52 58.42))
     (stroke (width 0) (type default))
   )
@@
   )
   (wire (pts (xy 44.45 91.44) (xy 44.45 96.52))
+    (stroke (width 0) (type default))
+  )
+  (wire (pts (xy 106.68 27.94) (xy 106.68 30.48))
     (stroke (width 0) (type default))
   )
@@
   (symbol (lib_id "Device:C") (at 44.45 148.59 0) (unit 1)
     (in_bom yes) (on_board yes) (dnp no) (fields_autoplaced)
-    (property "Reference" "C5" (at 48.26 147.955 0)
+    (property "Reference" "C6" (at 48.26 147.955 0)
       (effects (font (size 1.27 1.27)) (justify left))
     )
@@
       (project "button-debouncer"
         (path "/0f436cbe-229c-4c4e-a045-3abc4823e758"
-          (reference "C5") (unit 1)
+          (reference "C6") (unit 1)
         )
       )
@@
     )
   )
+  (symbol (lib_id "power:PWR_FLAG") (at 106.68 57.15 0) (unit 1)
+    (in_bom yes) (on_board yes) (dnp no) (fields_autoplaced)
+    (property "Reference" "#FLG02" (at 106.68 55.245 0)
+      (effects (font (size 1.27 1.27)) hide)
+    )
+    (property "Value" "PWR_FLAG" (at 106.68 53.34 0)
+      (effects (font (size 1.27 1.27)))
+    )
+    (property "Footprint" "" (at 106.68 57.15 0)
+      (effects (font (size 1.27 1.27)) hide)
+    )
+    (property "Datasheet" "~" (at 106.68 57.15 0)
+      (effects (font (size 1.27 1.27)) hide)
+    )
+    (pin "1")
+    (instances
+      (project "button-debouncer"
+        (path "/0f436cbe-229c-4c4e-a045-3abc4823e758"
+          (reference "#FLG02") (unit 1)
+        )
+      )
+    )
+  )
   (symbol (lib_id "4xxx:40106") (at 152.4 140.97 0) (unit 6)
     (in_bom yes) (on_board yes) (dnp no) (fields_autoplaced)
@@
   (symbol (lib_id "Device:C") (at 115.57 148.59 0) (unit 1)
     (in_bom yes) (on_board yes) (dnp no) (fields_autoplaced)
-    (property "Reference" "C7" (at 119.38 147.955 0)
+    (property "Reference" "C8" (at 119.38 147.955 0)
       (effects (font (size 1.27 1.27)) (justify left))
     )
@@
       (project "button-debouncer"
         (path "/0f436cbe-229c-4c4e-a045-3abc4823e758"
-          (reference "C7") (unit 1)
+          (reference "C8") (unit 1)
         )
       )
@@
   (symbol (lib_id "Device:C") (at 44.45 104.14 0) (unit 1)
     (in_bom yes) (on_board yes) (dnp no) (fields_autoplaced)
-    (property "Reference" "C3" (at 48.26 103.505 0)
+    (property "Reference" "C5" (at 48.26 103.505 0)
       (effects (font (size 1.27 1.27)) (justify left))
     )
@@
       (project "button-debouncer"
         (path "/0f436cbe-229c-4c4e-a045-3abc4823e758"
-          (reference "C3") (unit 1)
+          (reference "C5") (unit 1)
         )
       )
@@
     )
   )
+  (symbol (lib_id "power:PWR_FLAG") (at 106.68 27.94 0) (unit 1)
+    (in_bom yes) (on_board yes) (dnp no) (fields_autoplaced)
+    (property "Reference" "#FLG01" (at 106.68 26.035 0)
+      (effects (font (size 1.27 1.27)) hide)
+    )
+    (property "Value" "PWR_FLAG" (at 106.68 24.13 0)
+      (effects (font (size 1.27 1.27)))
+    )
+    (property "Footprint" "" (at 106.68 27.94 0)
+      (effects (font (size 1.27 1.27)) hide)
+    )
+    (property "Datasheet" "~" (at 106.68 27.94 0)
+      (effects (font (size 1.27 1.27)) hide)
+    )
+    (pin "1")
+    (instances
+      (project "button-debouncer"
+        (path "/0f436cbe-229c-4c4e-a045-3abc4823e758"
+          (reference "#FLG01") (unit 1)
+        )
+      )
+    )
+  )
   (symbol (lib_id "power:GND") (at 115.57 154.94 0) (mirror y) (unit 1)
     (in_bom yes) (on_board yes) (dnp no) (fields_autoplaced)
@@
   (symbol (lib_id "Device:C") (at 115.57 104.14 0) (unit 1)
     (in_bom yes) (on_board yes) (dnp no) (fields_autoplaced)
-    (property "Reference" "C6" (at 119.38 103.505 0)
+    (property "Reference" "C7" (at 119.38 103.505 0)
       (effects (font (size 1.27 1.27)) (justify left))
     )
@@
       (project "button-debouncer"
         (path "/0f436cbe-229c-4c4e-a045-3abc4823e758"
-          (reference "C6") (unit 1)
+          (reference "C7") (unit 1)
         )
       )
@@
   (symbol (lib_id "Device:C") (at 186.69 44.45 0) (unit 1)
     (in_bom yes) (on_board yes) (dnp no) (fields_autoplaced)
-    (property "Reference" "C8" (at 190.5 43.815 0)
+    (property "Reference" "C4" (at 190.5 43.815 0)
       (effects (font (size 1.27 1.27)) (justify left))
     )
@@
       (project "button-debouncer"
         (path "/0f436cbe-229c-4c4e-a045-3abc4823e758"
-          (reference "C8") (unit 1)
+          (reference "C4") (unit 1)
         )
       )
@@
   (symbol (lib_id "Device:C") (at 154.94 44.45 0) (unit 1)
     (in_bom yes) (on_board yes) (dnp no) (fields_autoplaced)
-    (property "Reference" "C4" (at 158.75 43.815 0)
+    (property "Reference" "C3" (at 158.75 43.815 0)
       (effects (font (size 1.27 1.27)) (justify left))
     )
@@
       (project "button-debouncer"
         (path "/0f436cbe-229c-4c4e-a045-3abc4823e758"
-          (reference "C4") (unit 1)
-        )
-      )
+          (reference "C3") (unit 1)
+        )
+      )

Commit message: added footprints to components
Parts:
- removed C2, C9: 1u, symbol Device:C
- removed J2, J4: Conn_01x02, symbol Connector_Generic:Conn_01x02
- removed SW3: SW_SPDT, symbol Switch:SW_SPDT
- added SW5: SW_SPDT, Button_Switch_THT:SW_Slide_1P2T_CK_OS102011MS2Q, symbol Switch:SW_SPDT
- C1: footprint (none) -> Capacitor_SMD:CP_Elec_4x4.5
- C3, C4: footprint (none) -> Capacitor_SMD:C_0805_2012Metric
- C5, C6, C7, C8: footprint (none) -> Capacitor_SMD:C_0402_1005Metric
- D1, D2, D3, D4: footprint (none) -> LED_SMD:LED_0402_1005Metric
- H1, H2, H3, H4: footprint (none) -> MountingHole:MountingHole_2.5mm_Pad
- J1: footprint (none) -> Connector_PinHeader_2.54mm:PinHeader_1x02_P2.54mm_Vertical
- J2: renamed from J3; footprint (none) -> Connector_PinHeader_2.54mm:PinHeader_1x02_P2.54mm_Vertical
- J3: renamed from J5; footprint (none) -> Connector_PinSocket_2.54mm:PinSocket_1x06_P2.54mm_Vertical
- R1, R10, R11, R12, R2, R3, R4, R5, R6, R7, R8, R9: footprint (none) -> Resistor_SMD:R_0402_1005Metric
- SW1, SW2: footprint (none) -> Button_Switch_THT:SW_PUSH_6mm
- SW3: renamed from SW4; footprint (none) -> Button_Switch_THT:SW_PUSH_6mm
- SW4: renamed from SW5; footprint (none) -> Button_Switch_THT:SW_PUSH_6mm
- SW6: footprint (none) -> Button_Switch_THT:SW_Slide_1P2T_CK_OS102011MS2Q
- U1, U2: footprint (none) -> Package_SO:SOIC-14_3.9x8.7mm_P1.27mm
Connections:
- net Q1: now also U1.8; no longer U1.2
- net Q2: now also U1.6; no longer U1.4
- net Q3: now also SW5.2 (B)
- net at C6.1, R3.2, R4.2: now also U1.5; no longer U1.3
- net at C7.1, R5.2, R6.2: now also U1.3; no longer U1.5
- net at C5.1, R1.2, R2.2: now also U1.9; no longer U1.1
- net at U1.12: now also SW6.3 (C); no longer SW6.1 (A)
- net at C8.1, R7.2, R8.2: now also U1.1; no longer U1.11
- new net: SW5.1 (A), U1.11, U1.4
- new net: SW6.1 (A), U1.13, U1.2
- new net: SW5.3 (C), U1.10
Other:
- moved on the sheet: C1, J3

Commit message: updated resistors values
Parts:
- R1, R3, R5, R7: value R -> 100
- R10, R11, R12, R9: value R -> 330
- R2, R4, R6, R8: value R -> 10k
Changed lines of the file:
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@@
       (effects (font (size 1.27 1.27)))
     )
-    (property "Value" "R" (at 245.11 45.72 90)
+    (property "Value" "330" (at 245.11 45.72 90)
       (effects (font (size 1.27 1.27)))
     )
@@
       (effects (font (size 1.27 1.27)))
     )
-    (property "Value" "R" (at 35.56 93.98 90)
+    (property "Value" "100" (at 35.56 93.98 90)
       (effects (font (size 1.27 1.27)))
     )
@@
       (effects (font (size 1.27 1.27)) (justify left))
     )
-    (property "Value" "R" (at 46.99 133.985 0)
+    (property "Value" "10k" (at 46.99 133.985 0)
       (effects (font (size 1.27 1.27)) (justify left))
     )
@@
       (effects (font (size 1.27 1.27)))
     )
-    (property "Value" "R" (at 245.11 59.69 90)
+    (property "Value" "330" (at 245.11 59.69 90)
       (effects (font (size 1.27 1.27)))
     )
@@
       (effects (font (size 1.27 1.27)) (justify left))
     )
-    (property "Value" "R" (at 118.11 133.985 0)
+    (property "Value" "10k" (at 118.11 133.985 0)
       (effects (font (size 1.27 1.27)) (justify left))
     )
@@
       (effects (font (size 1.27 1.27)))
     )
-    (property "Value" "R" (at 106.68 93.98 90)
+    (property "Value" "100" (at 106.68 93.98 90)
       (effects (font (size 1.27 1.27)))
     )
@@
       (effects (font (size 1.27 1.27)))
     )
-    (property "Value" "R" (at 35.56 138.43 90)
+    (property "Value" "100" (at 35.56 138.43 90)
       (effects (font (size 1.27 1.27)))
     )
@@
       (effects (font (size 1.27 1.27)))
     )
-    (property "Value" "R" (at 106.68 138.43 90)
+    (property "Value" "100" (at 106.68 138.43 90)
       (effects (font (size 1.27 1.27)))
     )
@@
       (effects (font (size 1.27 1.27)) (justify left))
     )
-    (property "Value" "R" (at 46.99 89.535 0)
+    (property "Value" "10k" (at 46.99 89.535 0)
       (effects (font (size 1.27 1.27)) (justify left))
     )
@@
       (effects (font (size 1.27 1.27)) (justify left))
     )
-    (property "Value" "R" (at 118.11 89.535 0)
+    (property "Value" "10k" (at 118.11 89.535 0)
       (effects (font (size 1.27 1.27)) (justify left))
     )
@@
       (effects (font (size 1.27 1.27)))
     )
-    (property "Value" "R" (at 245.11 31.75 90)
+    (property "Value" "330" (at 245.11 31.75 90)
       (effects (font (size 1.27 1.27)))
     )
@@
       (effects (font (size 1.27 1.27)))
     )
-    (property "Value" "R" (at 245.11 73.66 90)
-      (effects (font (size 1.27 1.27)))
-    )
+    (property "Value" "330" (at 245.11 73.66 90)
+      (effects (font (size 1.27 1.27)))
+    )
