File: Project/button-debouncer.kicad_pcb (KiCad board)
At the start: 2 copper layers, 40 x 50 mm, 38 parts, among them J1 Conn_01x02, J2 Conn_01x02, J3 Conn_01x06, SW1 SW_Push, SW2 SW_Push, SW3 SW_Push, SW4 SW_Push, SW5 SW_SPDT, SW6 SW_SPDT, U1 40106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

Commit message: project in stable version - production ordered
Parts:
- R1, R3, R5, R7: value R -> 100
- R10, R11, R12, R9: value R -> 330
- R2, R4, R6, R8: value R -> 10k
Changed lines of the file:
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@@
       (outputformat 1)
       (mirror false)
-      (drillshape 1)
+      (drillshape 0)
       (scaleselection 1)
       (outputdirectory "")
@@
         (effects (font (size 1 1) (thickness 0.15)))
     )
-    (fp_text value "R" (at 0 1.17 90) (layer "F.Fab")
+    (fp_text value "330" (at 0 1.17 90) (layer "F.Fab")
         (effects (font (size 1 1) (thickness 0.15)))
     )
@@
         (effects (font (size 1 1) (thickness 0.15)))
     )
-    (fp_text value "R" (at 0 1.17) (layer "F.Fab")
+    (fp_text value "100" (at 0 1.17) (layer "F.Fab")
         (effects (font (size 1 1) (thickness 0.15)))
     )
@@
         (effects (font (size 1 1) (thickness 0.15)))
     )
-    (fp_text value "R" (at 0 1.17) (layer "F.Fab")
+    (fp_text value "10k" (at 0 1.17) (layer "F.Fab")
         (effects (font (size 1 1) (thickness 0.15)))
     )
@@
         (effects (font (size 1 1) (thickness 0.15)))
     )
-    (fp_text value "R" (at 0 1.17) (layer "F.Fab")
+    (fp_text value "10k" (at 0 1.17) (layer "F.Fab")
         (effects (font (size 1 1) (thickness 0.15)))
     )
@@
         (effects (font (size 1 1) (thickness 0.15)))
     )
-    (fp_text value "R" (at 0 1.17) (layer "F.Fab")
+    (fp_text value "10k" (at 0 1.17) (layer "F.Fab")
         (effects (font (size 1 1) (thickness 0.15)))
     )
@@
         (effects (font (size 1 1) (thickness 0.15)))
     )
-    (fp_text value "R" (at 0 1.17 90) (layer "F.Fab")
+    (fp_text value "330" (at 0 1.17 90) (layer "F.Fab")
         (effects (font (size 1 1) (thickness 0.15)))
     )
@@
         (effects (font (size 1 1) (thickness 0.15)))
     )
-    (fp_text value "R" (at 0 1.17) (layer "F.Fab")
+    (fp_text value "100" (at 0 1.17) (layer "F.Fab")
         (effects (font (size 1 1) (thickness 0.15)))
     )
@@
         (effects (font (size 1 1) (thickness 0.15)))
     )
-    (fp_text value "R" (at 0 1.17 90) (layer "F.Fab")
+    (fp_text value "330" (at 0 1.17 90) (layer "F.Fab")
         (effects (font (size 1 1) (thickness 0.15)))
     )
@@
         (effects (font (size 1 1) (thickness 0.15)))
     )
-    (fp_text value "R" (at 0 1.17) (layer "F.Fab")
+    (fp_text value "10k" (at 0 1.17) (layer "F.Fab")
         (effects (font (size 1 1) (thickness 0.15)))
     )
@@
         (effects (font (size 1 1) (thickness 0.15)))
     )
-    (fp_text value "R" (at 0 1.17) (layer "F.Fab")
+    (fp_text value "100" (at 0 1.17) (layer "F.Fab")
         (effects (font (size 1 1) (thickness 0.15)))
     )
@@
         (effects (font (size 1 1) (thickness 0.15)))
     )
-    (fp_text value "R" (at 0 1.17) (layer "F.Fab")
+    (fp_text value "100" (at 0 1.17) (layer "F.Fab")
         (effects (font (size 1 1) (thickness 0.15)))
     )
@@
         (effects (font (size 1 1) (thickness 0.15)))
     )
-    (fp_text value "R" (at 0 1.17 90) (layer "F.Fab")
-        (effects (font (size 1 1) (thickness 0.15)))
-    )
+    (fp_text value "330" (at 0 1.17 90) (layer "F.Fab")
+        (effects (font (size 1 1) (thickness 0.15)))
+    )
